Commit message: Frame trans ok, rotation wrong

File: robot_urdf/urdf/uam_urdf.urdf (robot description, URDF)
Before this commit: robot uam_urdf, 9 links, 8 joints
Links:
- link uav_link: mass 0.354035 -> None
Joints:
- joint fixed_joint_0: origin xyz=0 0 0.07 rpy=0 0 0 -> xyz=0 0 0.07 rpy=3.1416 -1.5708 0

Commit message: tasks done under vicon 1213

File: robot_urdf/urdf/uam_urdf.urdf (robot description, URDF)
Before this commit: robot uam_urdf, 9 links, 8 joints
Joints:
- joint fixed_joint_0: origin xyz=0 0 0.07 rpy=3.1416 -1.5708 0 -> xyz=0 0 0.03 rpy=3.1416 -1.5708 0
- joint revolute_joint_3: limit lower=-2.618 upper=2.618 effort=1000.0 velocity=0.5 -> lower=-6.28 upper=6.28 effort=1000.0 velocity=0.5
- joint revolute_joint_5: limit lower=-2.618 upper=2.618 effort=1000.0 velocity=0.5 -> lower=-6.28 upper=6.28 effort=1000.0 velocity=0.5; origin xyz=0.02085 0.0017632 0 rpy=1.5708 0 1.5708 -> xyz=0.02085 0.0067632 0 rpy=1.5708 0 1.5708

File: robot_urdf/urdf/uav2.urdf (robot description, URDF)
Before this commit: robot robot_urdf, 8 links, 7 joints
Joints:
- joint revolute_joint_3: limit lower=-2.618 upper=2.618 effort=1000.0 velocity=0.5 -> lower=-6.28 upper=6.28 effort=1000.0 velocity=0.5
- joint revolute_joint_4: limit lower=-2.618 upper=2.618 effort=1000.0 velocity=0.5 -> lower=-1.57 upper=1.57 effort=1000.0 velocity=0.5
- joint revolute_joint_5: limit lower=-2.618 upper=2.618 effort=1000.0 velocity=0.5 -> lower=-6.28 upper=6.28 effort=1000.0 velocity=0.5
